Commit message: Moved env_controllers, utils update, cartpole updates, various fixes, controlledEnv can not do more controller steps in one env step, simple_camera args fix

File: src/lr_gym/models/simple_camera.sdf.xacro (robot description, xacro)
@@ -1,7 +1,12 @@
 <?xml version="1.0" ?>
 <sdf version="1.5" xmlns:xacro="http://www.ros.org/wiki/xacro">
-  <xacro:property name="camera_width" value="1920" />
-  <xacro:property name="camera_height" value="1080" />
-  <model name="box">
+  <xacro:arg name="camera_width" default="1920"/>
+  <xacro:arg name="camera_height" default="1080"/>
+  <xacro:arg name="frame_rate" default="30"/>
+  <xacro:property name="camera_width" value="$(arg camera_width)" />
+  <xacro:property name="camera_height" value="$(arg camera_height)" />
+  <xacro:property name="frame_rate" value="$(arg frame_rate)" />
+  <model name="camera_model">
+    <static>true</static>
     <link name="simple_camera_link">
         <sensor type="camera" name="simple_camera">
@@ -18,6 +23,7 @@
           </camera>
           <always_on>1</always_on>
-          <update_rate>30</update_rate>
+          <update_rate>${frame_rate}</update_rate>
           <visualize>true</visualize>
+          <topic>simple_camera</topic>
         </sensor>
     </link>

Commit message: getRenderings should now return a dict, pybullet cameras work, many pybullet enhancements, many smaller things

File: src/lr_gym/models/simple_camera.sdf.xacro (robot description, xacro)
@@ -1,14 +1,18 @@
 <?xml version="1.0" ?>
-<sdf version="1.5" xmlns:xacro="http://www.ros.org/wiki/xacro">
+<sdf version="1.10" xmlns:xacro="http://www.ros.org/wiki/xacro">
   <xacro:arg name="camera_width" default="1920"/>
   <xacro:arg name="camera_height" default="1080"/>
   <xacro:arg name="frame_rate" default="30"/>
+  <xacro:arg name="camera_name"  default="simple_camera"/>
+  <xacro:arg name="camera_topic" default="$(arg camera_name)"/>
   <xacro:property name="camera_width" value="$(arg camera_width)" />
   <xacro:property name="camera_height" value="$(arg camera_height)" />
   <xacro:property name="frame_rate" value="$(arg frame_rate)" />
-  <model name="camera_model">
+  <xacro:property name="camera_topic" value="$(arg camera_topic)" />
+  <xacro:property name="camera_name" value="$(arg camera_name)" />
+  <model name="${camera_name}">
     <static>true</static>
     <link name="simple_camera_link">
-        <sensor type="camera" name="simple_camera">
+        <sensor type="camera" name="${camera_name}">
           <camera>
             <horizontal_fov>${69.4*3.14159/180}</horizontal_fov>
@@ -25,5 +29,5 @@
           <update_rate>${frame_rate}</update_rate>
           <visualize>true</visualize>
-          <topic>simple_camera</topic>
+          <topic>${camera_topic}</topic>
         </sensor>
         <inertial>
