Commit message: Cameras in PyBullet

File: src/lr_gym/models/cartpole_v0.urdf.xacro (robot description, xacro)
@@ -152,4 +152,5 @@
 		<dynamics damping="0.0" friction="${rail_friction}"/>
        	<limit lower="-2.0" upper="2.0" effort="2000000" velocity="100000"/>
+        <axis xyz="1 0 0"/>
 	</joint>
 	<joint name="fixed" type="fixed">

File: src/lr_gym/models/simple_camera.sdf.xacro (robot description, xacro)
@@ -27,5 +27,21 @@
           <topic>simple_camera</topic>
         </sensor>
+        <inertial>
+          <inertia>
+            <ixx>0</ixx>
+            <ixy>0</ixy>
+            <ixz>0</ixz>
+            <iyy>0</iyy>
+            <iyz>0</iyz>
+            <izz>0</izz>
+          </inertia>
+          <mass>0.0</mass>
+        </inertial>
     </link>
+    <!-- <link name="world"/>
+    <joint name="fixed" type="fixed">
+      <parent link="world"/>
+      <child link="simple_camera_link"/>
+    </joint> -->
   </model>
 </sdf>

Commit message: general updates, experimenting with mjx

File: src/lr_gym/models/cartpole_v0.urdf.xacro (robot description, xacro)
@@ -58,5 +58,5 @@
     <link name="world"/>
 	<link name="bar_link">
-		<visual>
+		<visual name = "bar_link_v">
 			<origin xyz="0 0 ${bar_height/2}" rpy="0 0 0"/>
 			<geometry>
@@ -64,5 +64,5 @@
 			</geometry>
 	   </visual>
-		<collision>
+		<collision name = "bar_link_c">
 			<origin xyz="0 0 ${bar_height/2}" rpy="0 0 0"/>
 			<geometry>
@@ -73,5 +73,5 @@
 	</link>
 	<gazebo reference="bar_link">
-		<visual name="visual">
+		<visual name="bar_link_v">
 			<material>
 			<ambient>$(arg bar_color)</ambient>
@@ -113,5 +113,5 @@
 	<link name="foot_link">
 		<origin xyz="${rail_x} ${rail_y} ${rail_z}" rpy="${rail_roll} ${rail_pitch} ${rail_yaw}"/>
-		<visual>
+		<visual name = "foot_link_v">
 			<origin xyz="0 0 ${rail_height/2}" rpy="0 0 0"/>
 			<geometry>
@@ -119,5 +119,5 @@
 			</geometry>
 	   </visual>
-  		<collision>
+  		<collision name = "foot_link_c">
 			<origin xyz="0 0 ${rail_height/2}" rpy="0 0 0"/>
 			<geometry>
