Commit message: Fixes for vec logger and rewards logging, threnderer and some 2d collision utils, imporvements in async_vec_env, robot_helper

File: src/adarl/models/cube.urdf (robot description, URDF)
Before this commit: robot cube, 2 links, 1 joints
Links:
- added link cube_link2; collision box size=1 1 1; visual box size=1 1 1
Joints:
- added joint joint2: type revolute, parent cube_link, child cube_link2, origin xyz=0 0 1 rpy=0 0 0, limit lower=-3.14159 upper=3.14159 effort=30 velocity=10.0
