Commit message: started working on vec adapters and mjx

File: src/adarl/models/hopper_v1.urdf.xacro (robot description, xacro)
@@ -34,5 +34,5 @@
   <xacro:property name="foot_position_z" value="0" />
   <xacro:property name="foot_orientation" value="0 1.570795 0" />
-  <xacro:property name="max_effort" value="1000" />
+  <xacro:property name="max_effort" value="100" />
   <xacro:property name="spawn_height" value="0.001" />
   <xacro:property name="gear" value="200" />
@@ -301,5 +301,5 @@
     </actuator>
   </transmission>
-  <link name="camera_link"/>
+  <!-- <link name="camera_link"/>
   <joint name="camera_joint" type="fixed">
     <origin xyz="0 -2.5 0.75" rpy="0 0 1.5707" />
@@ -334,4 +334,4 @@
         <visualize>0</visualize>
     </sensor>
-  </gazebo>
+  </gazebo> -->
 </robot>
