Commit message: implementing mjxadapter

File: src/adarl/models/cartpole_v0.urdf.xacro (robot description, xacro)
@@ -158,3 +158,10 @@
         <child link="foot_link"/>
     </joint>
+	<sensor name="my_camera_sensor" update_rate="20">
+		<parent link="world"/>
+		<origin xyz="0 2 0" rpy="0 0 -1.57"/>
+		<camera>
+			<image width="640" height="480" hfov="1.5708" format="RGB8" near="0.01" far="50.0"/>
+		</camera>
+	</sensor>
 </robot>

Commit message: setLinkState works

File: src/adarl/models/cartpole_v0.urdf.xacro (robot description, xacro)
@@ -158,10 +158,3 @@
         <child link="foot_link"/>
     </joint>
-	<sensor name="my_camera_sensor" update_rate="20">
-		<parent link="world"/>
-		<origin xyz="0 2 0" rpy="0 0 -1.57"/>
-		<camera>
-			<image width="640" height="480" hfov="1.5708" format="RGB8" near="0.01" far="50.0"/>
-		</camera>
-	</sensor>
 </robot>

File: src/adarl/models/cubes.urdf (robot description, URDF)
Before this commit: robot cube, 3 links, 2 joints
Links:
- removed link cube_link
- added link cube_link1, mass 1; collision box size=1 1 1; visual box size=1 1 1
- link cube_link2: mass None -> 1
Joints:
- removed joint fixed
- added joint joint1: type revolute, parent world, child cube_link1, origin xyz=0 0 1 rpy=0 0 0, limit lower=-3.14159 upper=3.14159 effort=30 velocity=10.0
- joint joint2: origin xyz=0 0 1 rpy=0 0 0 -> xyz=0 0 0 rpy=0 0 0; parent cube_link -> world

File: src/adarl/models/simple_camera.mjcf.xacro (robot description, xacro)
@@ -3,11 +3,17 @@
   <xacro:arg name="camera_height" default="1080"/>
   <xacro:arg name="camera_name"  default="simple_camera"/>
+  <xacro:arg name="position_xyz"  default="0 0 0"/>
+  <xacro:arg name="orientation_wxyz"  default="1 0 0 0"/>
   <xacro:property name="camera_width" value="$(arg camera_width)" />
   <xacro:property name="camera_height" value="$(arg camera_height)" />
   <xacro:property name="camera_name" value="$(arg camera_name)" />
+  <xacro:property name="position_xyz" value="$(arg position_xyz)" />
+  <xacro:property name="orientation_wxyz" value="$(arg orientation_wxyz)" />
+    <compiler angle="radian"/>
     <worldbody>
-        <body name="simple_camera_link">
+        <body name="simple_camera_link" pos="${position_xyz}"  quat="${orientation_wxyz}">
+        <!-- xyaxes="-1 0 0 0 0 1"> -->
           <camera name="${camera_name}"
-                  fovy="${69.4*3.14159/180*camera_height/camera_width}"
+                  fovy="${70*camera_height/camera_width}"
                   resolution="${camera_width} ${camera_height}"
           />

Commit message: updates for dvae-sac

File: src/adarl/models/cartpole_v0.urdf.xacro (robot description, xacro)
@@ -1,14 +1,14 @@
 <?xml version="1.0" encoding="utf-8"  ?>
 <robot name="cartpole_v0" xmlns:xacro="http://www.ros.org/wiki/xacro">
-	<xacro:arg name="bar_width" default="0.05" />
+	<xacro:arg name="bar_width" default="0.1" />
 	<xacro:arg name="bar_length" default="0.05" />
 	<xacro:arg name="bar_height" default="0.8" />
 	<xacro:arg name="bar_mass" default="1" />
-	<xacro:arg name="bar_color" default="1 0.5088 0.0468 1" /> <!-- Orange -->
+	<xacro:arg name="bar_color" default="1 0.7 0.1 1" /> <!-- Orange -->
 	<xacro:arg name="base_width" default="0.4" />
 	<xacro:arg name="base_length" default="0.2" />
 	<xacro:arg name="base_height" default="0.2" />
 	<xacro:arg name="base_mass" default="2.5" />
-	<xacro:arg name="base_color" default="0 0 0 1" /> <!-- Black -->
+	<xacro:arg name="base_color" default="0.5 0.5 0.5 1" /> <!-- grey -->
 	<xacro:arg name="rail_color" default="1 1 1 1" /> <!-- White -->
 	<xacro:arg name="rail_width" default="6" />
@@ -24,4 +24,5 @@
 	<xacro:arg name="rail_pitch" default="0.0" />
 	<xacro:arg name="rail_yaw" default="0.0" />
+	<xacro:arg name="use_collisions" default="true" />
 	<xacro:property name="bar_width" default="$(arg bar_width)" />
 	<xacro:property name="bar_length" default="$(arg bar_length)" />
@@ -47,4 +48,5 @@
 	<xacro:property name="rail_pitch" default="$(arg rail_pitch)" />
 	<xacro:property name="rail_yaw" default="$(arg rail_yaw)" />
+	<xacro:property name="use_collisions" default="$(arg use_collisions)" />
 	<xacro:macro name="box_inertial" params="mass x y z pose_xyz pose_rpy">
 		<inertial>
@@ -63,11 +65,16 @@
 				<box size="${bar_width} ${bar_length} ${bar_height}"/>
 			</geometry>
-	   </visual>
-		<collision name = "bar_link_c">
-			<origin xyz="0 0 ${bar_height/2}" rpy="0 0 0"/>
-			<geometry>
-				<box size="${bar_width} ${bar_length} ${bar_height}"/>
-			</geometry>
-	   </collision>
+            <material name="bar_material">
+                <color rgba="$(arg bar_color)"/>
+            </material>
+		</visual>
+		<xacro:if value="${use_collisions}">
+			<collision name = "bar_link_c">
+				<origin xyz="0 0 ${bar_height/2}" rpy="0 0 0"/>
+				<geometry>
+					<box size="${bar_width} ${bar_length} ${bar_height}"/>
+				</geometry>
+			</collision>
+		</xacro:if>
 		<xacro:box_inertial mass="${bar_mass}" x="${bar_width}" y="${bar_length}" z="${bar_height}" pose_xyz="0 0 ${bar_height/2}" pose_rpy="0 0 0"/>
 	</link>
@@ -90,11 +97,16 @@
 				<box size="${base_width} ${base_length} ${base_height}"/>
 			</geometry>
-	   </visual>
-  		<collision>
-			<origin xyz="0 0 ${base_height}" rpy="0 0 0"/>
-			<geometry>
-				<box size="${base_width} ${base_length} ${base_height}"/>
-			</geometry>
-	   </collision>
+            <material name="base_material">
+                <color rgba="$(arg base_color)"/>
+            </material>
+	   	</visual>
+		<xacro:if value="${use_collisions}">
+			<collision>
+				<origin xyz="0 0 ${base_height}" rpy="0 0 0"/>
+				<geometry>
+					<box size="${base_width} ${base_length} ${base_height}"/>
+				</geometry>
+			</collision>
+		</xacro:if>
 		<xacro:box_inertial mass="${base_mass}" x="${base_width}" y="${base_length}" z="${base_height}" pose_xyz="0 0 ${base_height}" pose_rpy="0 0 0"/>
 	</link>
@@ -118,11 +130,16 @@
 				<box size="${rail_width} ${rail_length} ${rail_height}"/>
 			</geometry>
+            <material name="rail_material">
+                <color rgba="$(arg rail_color)"/>
+            </material>
 	   </visual>
-  		<collision name = "foot_link_c">
-			<origin xyz="0 0 ${rail_height/2}" rpy="0 0 0"/>
-			<geometry>
-				<box size="${rail_width} ${rail_length} ${rail_height}"/>
-			</geometry>
-	   </collision>
+		<xacro:if value="${use_collisions}">
+			<collision name = "foot_link_c">
+				<origin xyz="0 0 ${rail_height/2}" rpy="0 0 0"/>
+				<geometry>
+					<box size="${rail_width} ${rail_length} ${rail_height}"/>
+				</geometry>
+			</collision>
+		</xacro:if>
 		<xacro:box_inertial mass="${rail_mass}" x="${rail_width}" y="${rail_length}" z="${rail_height}" pose_xyz="0 0 ${rail_height/2}" pose_rpy="0 0 0"/>
 	</link>
@@ -139,10 +156,10 @@
       	</visual>
     </gazebo>
- 	<joint name="cartpole_joint" type="revolute">
+ 	<joint name="cartpole_joint" type="continuous">
     	<parent link="base_link"/>
     	<child link="bar_link"/>
     	<origin xyz="0 0 0.32" rpy="0 0 0"/>
 		<dynamics damping="0.0" friction="${hinge_friction}"/>
-       	<limit lower="-1.57" upper="1.57" effort="1" velocity="100"/>
+       	<limit effort="1" velocity="100"/>
         <axis xyz="0 1 0"/>
 	</joint>

Commit message: debugging CartpoleContinuousVecEnv

File: src/adarl/models/cartpole_v0.urdf.xacro (robot description, xacro)
@@ -1,28 +1,30 @@
 <?xml version="1.0" encoding="utf-8"  ?>
 <robot name="cartpole_v0" xmlns:xacro="http://www.ros.org/wiki/xacro">
-	<xacro:arg name="bar_width" default="0.1" />
-	<xacro:arg name="bar_length" default="0.05" />
-	<xacro:arg name="bar_height" default="0.8" />
-	<xacro:arg name="bar_mass" default="1" />
-	<xacro:arg name="bar_color" default="1 0.7 0.1 1" /> <!-- Orange -->
-	<xacro:arg name="base_width" default="0.4" />
+	<xacro:arg name="bar_width"   default="0.1" />
+	<xacro:arg name="bar_length"  default="0.05" />
+	<xacro:arg name="bar_height"  default="0.8" />
+	<xacro:arg name="bar_mass"    default="1" />
+	<xacro:arg name="base_width"  default="0.4" />
 	<xacro:arg name="base_length" default="0.2" />
 	<xacro:arg name="base_height" default="0.2" />
-	<xacro:arg name="base_mass" default="2.5" />
-	<xacro:arg name="base_color" default="0.5 0.5 0.5 1" /> <!-- grey -->
-	<xacro:arg name="rail_color" default="1 1 1 1" /> <!-- White -->
-	<xacro:arg name="rail_width" default="6" />
+	<xacro:arg name="base_mass"   default="1" />
+	<xacro:arg name="rail_width"  default="6" />
 	<xacro:arg name="rail_length" default="0.025" />
 	<xacro:arg name="rail_height" default="0.1" />
-	<xacro:arg name="rail_mass" default="5" />
-	<xacro:arg name="hinge_friction" default="0.1" />
-	<xacro:arg name="rail_friction" default="0.0" />
+	<xacro:arg name="rail_mass"   default="100" />
+	<xacro:arg name="hinge_friction" default="0.01" />
+	<xacro:arg name="rail_friction"  default="0.01" />
+	<xacro:arg name="hinge_damping"  default="0.1" />
+	<xacro:arg name="rail_damping"   default="0.1" />
 	<xacro:arg name="rail_x" default="0.0" />
 	<xacro:arg name="rail_y" default="0.0" />
 	<xacro:arg name="rail_z" default="0.0" />
-	<xacro:arg name="rail_roll" default="0.0" />
+	<xacro:arg name="rail_roll"  default="0.0" />
 	<xacro:arg name="rail_pitch" default="0.0" />
-	<xacro:arg name="rail_yaw" default="0.0" />
+	<xacro:arg name="rail_yaw"   default="0.0" />
 	<xacro:arg name="use_collisions" default="true" />
+	<xacro:arg name="bar_color"  default="1.0 0.7 0.1 1" /> <!-- Orange -->
+	<xacro:arg name="base_color" default="0.5 0.5 0.5 1" /> <!-- grey -->
+	<xacro:arg name="rail_color" default="1   1   1   1" /> <!-- White -->
 	<xacro:property name="bar_width" default="$(arg bar_width)" />
 	<xacro:property name="bar_length" default="$(arg bar_length)" />
@@ -42,4 +44,6 @@
 	<xacro:property name="hinge_friction" default="$(arg hinge_friction)" />
 	<xacro:property name="rail_friction" default="$(arg rail_friction)" />
+	<xacro:property name="hinge_damping" default="$(arg hinge_damping)" />
+	<xacro:property name="rail_damping" default="$(arg rail_damping)" />
 	<xacro:property name="rail_x" default="$(arg rail_x)" />
 	<xacro:property name="rail_y" default="$(arg rail_y)" />
@@ -160,6 +164,6 @@
     	<child link="bar_link"/>
     	<origin xyz="0 0 0.32" rpy="0 0 0"/>
-		<dynamics damping="0.0" friction="${hinge_friction}"/>
-       	<limit effort="1" velocity="100"/>
+		<dynamics damping="${hinge_damping}" friction="${hinge_friction}"/>
+       	<limit effort="100" velocity="100"/>
         <axis xyz="0 1 0"/>
 	</joint>
@@ -167,6 +171,6 @@
     	<parent link="foot_link"/>
     	<child link="base_link"/>
-		<dynamics damping="0.0" friction="${rail_friction}"/>
-       	<limit lower="-2.0" upper="2.0" effort="2000000" velocity="100000"/>
+		<dynamics damping="${rail_damping}" friction="${rail_friction}"/>
+       	<limit lower="-2.0" upper="2.0" effort="100" velocity="100"/>
         <axis xyz="1 0 0"/>
 	</joint>
