Commit message: Add stereo camera presets; take a horizontal fov in the camera model
_STEREO_CAMERAS lists zedxmini2.2mm and zedxmini4mm with focal length in
pixels at the native width, baseline and depth range.
stereo_camera_params() builds StereoDepthSimParams for a given render
width, scaling the pixel-valued figures from the native width - focal
length, disparity noise, sub-pixel step, fattening, shadow and blob size
- and takes per-field overrides. stereo_camera_hfov_degrees() derives the
field of view from the same table.

simple_camera.mjcf.xacro takes horizontal_fov_degrees and converts it to
mujoco's vertical fovy through the image aspect ratio with atan/tan,
where before it rescaled 70 degrees linearly.

File: src/adarl/models/simple_camera.mjcf.xacro (robot description, xacro)
@@ -5,4 +5,5 @@
   <xacro:arg name="position_xyz"  default="0 0 0"/>
   <xacro:arg name="orientation_wxyz"  default="1 0 0 0"/>
+  <xacro:arg name="horizontal_fov_degrees" default="70.0"/>
   <xacro:property name="camera_width" value="$(arg camera_width)" />
   <xacro:property name="camera_height" value="$(arg camera_height)" />
@@ -10,4 +11,9 @@
   <xacro:property name="position_xyz" value="$(arg position_xyz)" />
   <xacro:property name="orientation_wxyz" value="$(arg orientation_wxyz)" />
+  <xacro:property name="horizontal_fov_degrees" value="$(arg horizontal_fov_degrees)" />
+  <!-- mujoco specifies the *vertical* fov: converted through the image aspect ratio. Not a linear
+       rescaling, which would be noticeably off for a wide lens. -->
+  <xacro:property name="fovy_degrees"
+                  value="${2*atan(tan(radians(horizontal_fov_degrees)/2)*camera_height/camera_width)*180/pi}" />
     <compiler angle="radian"/>
     <worldbody>
@@ -15,5 +21,5 @@
           <!-- Make it so that, in the camera_link frame, the camera looks toward x, with z pointing up and y left -->
           <camera name="${camera_name}"
-                  fovy="${70*camera_height/camera_width}"
+                  fovy="${fovy_degrees}"
                   resolution="${camera_width} ${camera_height}"
                   xyaxes="0 -1 0 0 0 1"
